Commit message: feat(taccap-gripper): enhance TacCap replay functionality and semantics
- Updated the handling of recorded `left_tcp` and `right_tcp` poses to treat them as canonical TCP by default, with an option to apply side-specific tracker-to-TCP transforms when selected.
- Improved the URDF loading process by ensuring both left and right URDFs define link4 with the same canonical orientation, preventing unintended rotations during playback.
- Introduced a new `TacCapPoseProfile` to manage pose corrections and metadata, allowing for more accurate trajectory playback and visualization.
- Enhanced the URDF viewer to support pose mode selection, providing users with clearer feedback on the current pose mode.
- Added tests to validate the new pose semantics and ensure correct functionality across various scenarios.

This update significantly improves the accuracy and usability of TacCap gripper data during 3D replay, enhancing the overall user experience in pose analysis.

File: public/urdf/taccap-grippers/left/gripper.urdf (robot description, URDF)
Before this commit: robot taccap_left_gripper, 5 links, 4 joints
Joints:
- joint joint4: origin xyz=0.164636788170065 0 -0.0158499715519367 rpy=0 0 -1.5707963267949 -> xyz=0.164636788170065 0 -0.0158499715519367 rpy=0 0 0
